File: board/MXKeyboard_RGB.brd (EAGLE design)
At the start: 433.1 x 135.9 mm, 363 parts, among them Q1 DMN65D8L, Q2 DMP2240UDM, U1 TLC5947RHBT, U10 TLC5947RHBT, U11 ATXMEGA256A3U-MH, U12 NTS0104, U14 TC1015-3.3VCT713, U15 74HC238BQ, U16 74HC238BQ, U17 74HC238BQ, U18 TLC5947RHBT, U19 TLC5947RHBT, U2 TLC5947RHBT, U20 TLC5947RHBT, U21 TLC5947RHBT, U22 TLC5947RHBT, U3 TLC5947RHBT, U4 TLC5947RHBT, U5 TLC5947RHBT, U6 TLC5947RHBT, U7 TLC5947RHBT, U8 TLC5947RHBT, U9 TLC5947RHBT

Commit message: Added some fixes for hardware borkage we've discovered
Connections:
- net +5V: now also LED71.2
Changed lines of the file:
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@@
 <attribute name="OC_FARNELL" value="2449455" x="420.37" y="107.315" size="1.778" layer="27" rot="R90" display="off"/>
 <attribute name="URL" value="http://uk.farnell.com/iqd-frequency-products/lfspxo025494/oscillator-16mhz-15pf-smd/dp/2449455" x="420.37" y="107.315" size="1.778" layer="27" rot="R90" display="off"/>
+<attribute name="ALT_OC_FARNELL" value="2854286" x="420.37" y="107.315" size="1.778" layer="27" rot="R90" display="off"/>
+<attribute name="ALT_URL" value="https://uk.farnell.com/multicomp/mcsjk-3n-16-00-3-3-25-b/oscillator-16mhz-3-2mm-x-2-5mm/dp/2854286" x="420.37" y="107.315" size="1.778" layer="27" rot="R90" display="off"/>
+<attribute name="ALT_MFR" value="Multicomp" x="420.37" y="107.315" size="1.778" layer="27" rot="R90" display="off"/>
+<attribute name="ALT_MPN" value="MCSJK-3N-16.00-3.3-25-B" x="420.37" y="107.315" size="1.778" layer="27" rot="R90" display="off"/>
 </element>
 <element name="U18" library="MXKeyboard" package="PVQFN32" value="TLC5947RHBT" x="76.835" y="101.6" smashed="yes" rot="R90">
@@
 <via x="391.16" y="122.682" extent="1-16" drill="0.3"/>
 <via x="391.16" y="121.412" extent="1-16" drill="0.3"/>
+<contactref element="LED71" pad="2"/>
 </signal>
 <signal name="EARTH_USB">
