File: board/Key_matrix.sch (KiCad schematic (older format))
At the start: 155 parts

Commit message: Added a 1.25 unit key to the library and swapepd the home keys about so they're now the 6.25u spacebar layout
Parts:
- S12, S61, S67: footprint MXKeyboard_RGB:MX_KEY_NORM -> MXKeyboard_RGB:MX_KEY_1.25u
- S18, S55, S6, S73: footprint MXKeyboard_RGB:MX_KEY_1.1 -> MXKeyboard_RGB:MX_KEY_1.25u
Changed lines of the file:
@@
 F 0 "S6" H 1900 5700 59  0000 L BNN
 F 1 "LCtrl" H 2300 5500 59  0000 R BNN
-F 2 "MXKeyboard_RGB:MX_KEY_1.1" H 2100 5600 50  0001 C CNN
+F 2 "MXKeyboard_RGB:MX_KEY_1.25u" H 2100 5600 50  0001 C CNN
 F 3 "" H 2100 5600 50  0001 C CNN
 	1    2100 5600
@@
 F 0 "S12" H 2700 5700 59  0000 L BNN
 F 1 "LMeta" H 3100 5500 59  0000 R BNN
-F 2 "MXKeyboard_RGB:MX_KEY_NORM" H 2900 5600 50  0001 C CNN
+F 2 "MXKeyboard_RGB:MX_KEY_1.25u" H 2900 5600 50  0001 C CNN
 F 3 "" H 2900 5600 50  0001 C CNN
 	1    2900 5600
@@
 F 0 "S18" H 3500 5700 59  0000 L BNN
 F 1 "LAlt" H 3900 5500 59  0000 R BNN
-F 2 "MXKeyboard_RGB:MX_KEY_1.1" H 3700 5600 50  0001 C CNN
+F 2 "MXKeyboard_RGB:MX_KEY_1.25u" H 3700 5600 50  0001 C CNN
 F 3 "" H 3700 5600 50  0001 C CNN
 	1    3700 5600
@@
 F 0 "S55" H 9100 5700 59  0000 L BNN
 F 1 "RAlt_Gr" H 9500 5500 59  0000 R BNN
-F 2 "MXKeyboard_RGB:MX_KEY_1.1" H 9300 5600 50  0001 C CNN
+F 2 "MXKeyboard_RGB:MX_KEY_1.25u" H 9300 5600 50  0001 C CNN
 F 3 "" H 9300 5600 50  0001 C CNN
 	1    9300 5600
@@
 F 0 "S61" H 9900 5700 59  0000 L BNN
 F 1 "RMeta" H 10300 5500 59  0000 R BNN
-F 2 "MXKeyboard_RGB:MX_KEY_NORM" H 10100 5600 50  0001 C CNN
+F 2 "MXKeyboard_RGB:MX_KEY_1.25u" H 10100 5600 50  0001 C CNN
 F 3 "" H 10100 5600 50  0001 C CNN
 	1    10100 5600
@@
 F 0 "S67" H 10700 5700 59  0000 L BNN
 F 1 "Menu" H 11100 5500 59  0000 R BNN
-F 2 "MXKeyboard_RGB:MX_KEY_NORM" H 10900 5600 50  0001 C CNN
+F 2 "MXKeyboard_RGB:MX_KEY_1.25u" H 10900 5600 50  0001 C CNN
 F 3 "" H 10900 5600 50  0001 C CNN
 	1    10900 5600
@@
 F 0 "S73" H 11500 5700 59  0000 L BNN
 F 1 "RCtrl" H 11900 5500 59  0000 R BNN
-F 2 "MXKeyboard_RGB:MX_KEY_1.1" H 11700 5600 50  0001 C CNN
+F 2 "MXKeyboard_RGB:MX_KEY_1.25u" H 11700 5600 50  0001 C CNN
 F 3 "" H 11700 5600 50  0001 C CNN
 	1    11700 5600

Commit message: Updated the footprints in the schematic having renamed all of my published libraries
Parts:
- R1, R2, R3, R30, R31, R32, R33, R34, R35, R4, R5, R6: footprint rcl:R0603 -> rhais_rcl:R0603
Changed lines of the file:
@@
 F 0 "R31" H 1250 4059 59  0000 L BNN
 F 1 "20k" H 1400 3930 59  0000 R TNN
-F 2 "rcl:R0603" H 1300 4000 50  0001 C CNN
+F 2 "rhais_rcl:R0603" H 1300 4000 50  0001 C CNN
 F 3 "" H 1300 4000 50  0001 C CNN
 F 4 "Multicomp" H 1300 4000 59  0001 L BNN "MFR"
@@
 F 0 "R32" H 1250 4359 59  0000 L BNN
 F 1 "20k" H 1400 4230 59  0000 R TNN
-F 2 "rcl:R0603" H 1300 4300 50  0001 C CNN
+F 2 "rhais_rcl:R0603" H 1300 4300 50  0001 C CNN
 F 3 "" H 1300 4300 50  0001 C CNN
 F 4 "Multicomp" H 1300 4300 59  0001 L BNN "MFR"
@@
 F 0 "R33" H 1250 4659 59  0000 L BNN
 F 1 "20k" H 1400 4530 59  0000 R TNN
-F 2 "rcl:R0603" H 1300 4600 50  0001 C CNN
+F 2 "rhais_rcl:R0603" H 1300 4600 50  0001 C CNN
 F 3 "" H 1300 4600 50  0001 C CNN
 F 4 "Multicomp" H 1300 4600 59  0001 L BNN "MFR"
@@
 F 0 "R34" H 1250 4959 59  0000 L BNN
 F 1 "20k" H 1400 4830 59  0000 R TNN
-F 2 "rcl:R0603" H 1300 4900 50  0001 C CNN
+F 2 "rhais_rcl:R0603" H 1300 4900 50  0001 C CNN
 F 3 "" H 1300 4900 50  0001 C CNN
 F 4 "Multicomp" H 1300 4900 59  0001 L BNN "MFR"
@@
 F 0 "R35" H 1250 5459 59  0000 L BNN
 F 1 "20k" H 1400 5330 59  0000 R TNN
-F 2 "rcl:R0603" H 1300 5400 50  0001 C CNN
+F 2 "rhais_rcl:R0603" H 1300 5400 50  0001 C CNN
 F 3 "" H 1300 5400 50  0001 C CNN
 F 4 "Multicomp" H 1300 5400 59  0001 L BNN "MFR"
@@
 F 0 "R2" V 20250 4000 59  0000 C BNN
 F 1 "20k" V 20350 4000 59  0000 C TNN
-F 2 "rcl:R0603" H 20300 4000 50  0001 C CNN
+F 2 "rhais_rcl:R0603" H 20300 4000 50  0001 C CNN
 F 3 "" H 20300 4000 50  0001 C CNN
 F 4 "Multicomp" H 20300 4000 59  0001 L BNN "MFR"
@@
 F 0 "R6" V 20250 5200 59  0000 C BNN
 F 1 "20k" V 20350 5200 59  0000 C TNN
-F 2 "rcl:R0603" H 20300 5200 50  0001 C CNN
+F 2 "rhais_rcl:R0603" H 20300 5200 50  0001 C CNN
 F 3 "" H 20300 5200 50  0001 C CNN
 F 4 "Multicomp" H 20300 5200 59  0001 L BNN "MFR"
@@
 F 0 "R5" V 20250 4900 59  0000 C BNN
 F 1 "20k" V 20350 4900 59  0000 C TNN
-F 2 "rcl:R0603" H 20300 4900 50  0001 C CNN
+F 2 "rhais_rcl:R0603" H 20300 4900 50  0001 C CNN
 F 3 "" H 20300 4900 50  0001 C CNN
 F 4 "Multicomp" H 20300 4900 59  0001 L BNN "MFR"
@@
 F 0 "R4" V 20250 4600 59  0000 C BNN
 F 1 "20k" V 20350 4600 59  0000 C TNN
-F 2 "rcl:R0603" H 20300 4600 50  0001 C CNN
+F 2 "rhais_rcl:R0603" H 20300 4600 50  0001 C CNN
 F 3 "" H 20300 4600 50  0001 C CNN
 F 4 "Multicomp" H 20300 4600 59  0001 L BNN "MFR"
@@
 F 0 "R3" V 20250 4300 59  0000 C BNN
 F 1 "20k" V 20350 4300 59  0000 C TNN
-F 2 "rcl:R0603" H 20300 4300 50  0001 C CNN
+F 2 "rhais_rcl:R0603" H 20300 4300 50  0001 C CNN
 F 3 "" H 20300 4300 50  0001 C CNN
 F 4 "Multicomp" H 20300 4300 59  0001 L BNN "MFR"
@@
 F 0 "R1" V 20250 3500 59  0000 C BNN
 F 1 "20k" V 20350 3500 59  0000 C TNN
-F 2 "rcl:R0603" H 20300 3500 50  0001 C CNN
+F 2 "rhais_rcl:R0603" H 20300 3500 50  0001 C CNN
 F 3 "" H 20300 3500 50  0001 C CNN
 F 4 "Multicomp" H 20300 3500 59  0001 L BNN "MFR"
@@
 F 0 "R30" H 1250 3559 59  0000 L BNN
 F 1 "20k" H 1400 3430 59  0000 R TNN
-F 2 "rcl:R0603" H 1300 3500 50  0001 C CNN
+F 2 "rhais_rcl:R0603" H 1300 3500 50  0001 C CNN
 F 3 "" H 1300 3500 50  0001 C CNN
 F 4 "Multicomp" H 1300 3500 59  0001 L BNN "MFR"
