File: board/Key_matrix.sch (KiCad schematic (older format))
At the start: 169 parts

Commit message: Renamed MXKeyboard_RGB => MXKeyboard and cleaned up the last of the old Eagle files we aren't using now
Parts:
- D1, D10, D11, D12, D13, D14, D15, D16, D17, D18, D19, D2, D20, D21, D22, D23, D24, D25, D26, D27, D28, D29, D3, D30, D31, D32, D33, D34, D35, D36, D37, D4, D5, D6, D7, D8, D9: symbol MXKeyboard_RGB-eagle-import:BAS16VY -> MXKeyboard-eagle-import:BAS16VY
- S1, S10, S100, S101, S102, S103, S104, S11, S13, S14, S15, S16, S17, S19, S2, S20, S21, S22, S23, S24, S25, S26, S27, S28, S29, S30, S31, S32, S33, S34, S35, S36, S37, S38, S40, S41, S42, S43, S44, S45, S46, S47, S48, S49, S50, S51, S52, S53, S54, S56, S57, S58, S59, S60, S62, S63, S64, S65, S66, S68, S69, S7, S70, S71, S76, S77, S78, S79, S8, S80, S81, S82, S83, S84, S85, S86, S87, S88, S89, S9, S90, S91, S92, S93, S95, S96, S97, S98, S99: footprint MXKeyboard_RGB:MX_KEY_NORM -> MXKeyboard:MX_KEY_NORM; symbol MXKeyboard_RGB-eagle-import:CHERRY_MX_KEY_NORM -> MXKeyboard-eagle-import:CHERRY_MX_KEY_NORM
- S105, S106: footprint MXKeyboard_RGB:MX_KEY_1.45X0.7 -> MXKeyboard:MX_KEY_1.45X0.7; symbol MXKeyboard_RGB-eagle-import:CHERRY_MX_KEY_1.45X0.7 -> MXKeyboard-eagle-import:CHERRY_MX_KEY_1.45X0.7
- S12, S61, S67: footprint MXKeyboard_RGB:MX_KEY_1.25u -> MXKeyboard:MX_KEY_1.25u; symbol MXKeyboard_RGB-eagle-import:CHERRY_MX_KEY_NORM -> MXKeyboard-eagle-import:CHERRY_MX_KEY_NORM
- S18, S55, S6, S73: footprint MXKeyboard_RGB:MX_KEY_1.25u -> MXKeyboard:MX_KEY_1.25u; symbol MXKeyboard_RGB-eagle-import:CHERRY_MX_KEY_1.1 -> MXKeyboard-eagle-import:CHERRY_MX_KEY_1.1
- S3: footprint MXKeyboard_RGB:MX_KEY_1.1 -> MXKeyboard:MX_KEY_1.1; symbol MXKeyboard_RGB-eagle-import:CHERRY_MX_KEY_1.1 -> MXKeyboard-eagle-import:CHERRY_MX_KEY_1.1
- S39: footprint MXKeyboard_RGB:MX_KEY_4.45 -> MXKeyboard:MX_KEY_4.45; symbol MXKeyboard_RGB-eagle-import:CHERRY_MX_KEY_4.45 -> MXKeyboard-eagle-import:CHERRY_MX_KEY_4.45
- S4: footprint MXKeyboard_RGB:MX_KEY_1.3 -> MXKeyboard:MX_KEY_1.3; symbol MXKeyboard_RGB-eagle-import:CHERRY_MX_KEY_1.3 -> MXKeyboard-eagle-import:CHERRY_MX_KEY_1.3
- S5: footprint MXKeyboard_RGB:MX_KEY_1.25u -> MXKeyboard:MX_KEY_1.25u; symbol MXKeyboard_RGB-eagle-import:CHERRY_MX_KEY_0.9 -> MXKeyboard-eagle-import:CHERRY_MX_KEY_0.9
- S72: footprint MXKeyboard_RGB:MX_KEY_2 -> MXKeyboard:MX_KEY_2; symbol MXKeyboard_RGB-eagle-import:CHERRY_MX_KEY_2 -> MXKeyboard-eagle-import:CHERRY_MX_KEY_2
- S74, S94: footprint MXKeyboard_RGB:MX_KEY_0.7X1.45 -> MXKeyboard:MX_KEY_0.7X1.45; symbol MXKeyboard_RGB-eagle-import:CHERRY_MX_KEY_0.7X1.45 -> MXKeyboard-eagle-import:CHERRY_MX_KEY_0.7X1.45
- S75: footprint MXKeyboard_RGB:MX_KEY_ENTER -> MXKeyboard:MX_KEY_ENTER; symbol MXKeyboard_RGB-eagle-import:CHERRY_MX_KEY_ENTER -> MXKeyboard-eagle-import:CHERRY_MX_KEY_ENTER
- STB1, STB10, STB11, STB12, STB13, STB14, STB2, STB3, STB4, STB5, STB6, STB7, STB8, STB9: footprint MXKeyboard_RGB:MX_STABILISER -> MXKeyboard:MX_STABILISER; symbol MXKeyboard_RGB-eagle-import:Cherry_MX_Stabiliser -> MXKeyboard-eagle-import:Cherry_MX_Stabiliser

Commit message: Cleaned up the BOM and added all the missing BOM information I could find
Parts:
- D1, D10, D11, D12, D13, D14, D15, D16, D17, D18, D19, D2, D20, D21, D22, D23, D24, D25, D26, D27, D28, D29, D3, D30, D31, D32, D33, D34, D35, D36, D37, D4, D5, D6, D7, D8, D9: MFR (none) -> Nexperia; MPN (none) -> BAS16VY,115; OC_FARNELL (none) -> 8734240; URL_FARNELL (none) -> https://uk.farnell.com/nexperia/bas16vy-115/diode-switching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
- R1, R2, R3, R30, R31, R32, R33, R34, R35, R4, R5, R6: MPN MC0063W0603120K5 -> MCWR06X2002FTL; OC_FARNELL 2130963 -> 2446610; URL_FARNELL (none) -> https://uk.farnell.com/multicomp/mcwr06x2002ftl/res-20k-1-0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
- S1, S10, S100, S101, S102, S103, S104, S105, S106, S11, S12, S13, S14, S15, S16, S17, S18, S19, S2, S20, S21, S22, S23, S24, S25, S26, S27, S28, S29, S3, S30, S31, S32, S33, S34, S35, S36, S37, S38, S39, S4, S40, S41, S42, S43, S44, S45, S46, S47, S48, S49, S5, S50, S51, S52, S53, S54, S55, S56, S57, S58, S59, S6, S60, S61, S62, S63, S64, S65, S66, S67, S68, S69, S7, S70, S71, S72, S73, S74, S75, S76, S77, S78, S79, S8, S80, S81, S82, S83, S84, S85, S86, S87, S88, S89, S9, S90, S91, S92, S93, S94, S95, S96, S97, S98, S99: MFR (none) -> Cherry GmbH; MPN (none) -> MX1A-G1NA; OC_MOUSER (none) -> 540-MX1A-G1NA; URL_MOUSER (none) -> https://www.mouser.co.uk/ProductDetail/MX1A-G1NA
