File: board/Processor_+_comms.sch (KiCad schematic (older format))
At the start: 39 parts, among them U11 ATXMEGA256A3U-MH, U12 NTS0104, U14 TC1015-3.3VCT713

Commit message: Cleaned up and fixed some more of the capacitors that are using the old import schematic symbol
Parts:
- C1, C7, C8, C9: symbol MXKeyboard_RGB-eagle-import:C-EUC0603K -> Device:C_Small
Other:
- moved on the sheet: R17
Changed lines of the file:
@@
 	9600 5400 9500 5400
 Wire Wire Line
-	9500 5400 9500 6200
-Wire Wire Line
-	9500 6200 9500 6600
-Wire Wire Line
-	9500 6200 9700 6200
-Wire Wire Line
-	9700 6200 9950 6200
-Wire Wire Line
-	9950 6200 9950 6100
-Wire Wire Line
-	9700 6050 9700 6200
-Wire Wire Line
-	9300 5850 9300 6200
-Wire Wire Line
-	9300 6200 9500 6200
-Connection ~ 9500 6200
-Connection ~ 9700 6200
+	9500 5400 9500 6100
+Wire Wire Line
+	9500 6100 9500 6200
+Wire Wire Line
+	9500 6100 9700 6100
+Wire Wire Line
+	9700 6100 9950 6100
+Wire Wire Line
+	9950 6100 9950 6000
+Wire Wire Line
+	9700 6000 9700 6100
+Wire Wire Line
+	9300 5850 9300 6100
+Wire Wire Line
+	9300 6100 9500 6100
+Connection ~ 9500 6100
+Connection ~ 9700 6100
 Wire Wire Line
 	5700 7500 5700 7400
@@
 	14200 6800 14200 6900
 Wire Wire Line
-	14200 6900 14000 6900
-Wire Wire Line
-	14000 6900 14000 7100
-Wire Wire Line
-	14000 7100 14000 7400
-Wire Wire Line
-	14000 7400 14200 7400
-Wire Wire Line
-	14150 7100 14000 7100
-Wire Wire Line
-	14000 7400 14000 7500
-Connection ~ 14000 7100
-Connection ~ 14000 7400
+	14200 6900 14100 6900
+Wire Wire Line
+	14100 6900 14100 7100
+Wire Wire Line
+	14100 7100 14100 7400
+Wire Wire Line
+	14100 7400 14200 7400
+Wire Wire Line
+	14200 7100 14100 7100
+Wire Wire Line
+	14100 7400 14100 7500
+Connection ~ 14100 7100
+Connection ~ 14100 7400
 Wire Wire Line
 	12800 7200 12800 7300
@@
 	9950 5700 10050 5700
 Wire Wire Line
-	9700 5850 9700 5700
+	9700 5800 9700 5700
 Connection ~ 9950 5700
 Text Label 10050 5700 0    50   ~ 0
@@
 	4500 4100 4700 4100
 Wire Wire Line
-	12600 5500 12600 5600
-Wire Wire Line
-	12600 5600 12600 5800
-Wire Wire Line
-	12600 5600 12100 5600
-Wire Wire Line
-	12100 5600 12100 5700
-Connection ~ 12600 5600
+	12600 5600 12600 5700
+Wire Wire Line
+	12600 5700 12600 5800
+Wire Wire Line
+	12600 5700 12100 5700
+Wire Wire Line
+	12100 5700 12100 5800
+Connection ~ 12600 5700
 Wire Wire Line
 	8200 2000 8400 2000
@@
 	14400 6800 14400 6900
 Wire Wire Line
-	14400 6900 14600 6900
-Wire Wire Line
-	14600 6900 14600 7100
-Wire Wire Line
-	14600 7100 14600 7400
-Wire Wire Line
-	14600 7400 14400 7400
-Wire Wire Line
-	14450 7100 14600 7100
-Wire Wire Line
-	14600 6900 15000 6900
-Connection ~ 14600 7100
-Text Label 14700 6900 0    70   ~ 0
+	14400 6900 14500 6900
+Wire Wire Line
+	14500 6900 14500 7100
+Wire Wire Line
+	14500 7100 14500 7400
+Wire Wire Line
+	14500 7400 14400 7400
+Wire Wire Line
+	14400 7100 14500 7100
+Wire Wire Line
+	14500 6900 14600 6900
+Connection ~ 14500 7100
+Text Label 14600 6900 0    70   ~ 0
 EARTH_PS/2
-Connection ~ 14600 6900
+Connection ~ 14500 6900
 Wire Wire Line
 	14300 5800 14300 5600
@@
 	13000 5600 13000 5500
 Wire Wire Line
-	13500 5700 13500 5600
+	13500 5800 13500 5600
 Connection ~ 13000 5600
 Connection ~ 13500 5600
@@
 $EndComp
 $Comp
-L MXKeyboard_RGB-eagle-import:C-EUC0603K C1
+L Device:C_Small C1
 U 1 1 F1C90C04
 P 9950 5900
 AR Path="/F1C90C04" Ref="C1"  Part="1"
 AR Path="/5F5D6257/F1C90C04" Ref="C1"  Part="1"
-F 0 "C1" H 10010 5915 59  0000 L BNN
-F 1 "0.1uF" H 10010 5715 59  0000 L BNN
+F 0 "C1" H 10000 5950 59  0000 L BNN
+F 1 "0.1uF" H 10000 5850 59  0000 L TNN
 F 2 "rhais_rcl:C0603" H 9950 5900 50  0001 C CNN
 F 3 "" H 9950 5900 50  0001 C CNN
@@
 $EndComp
 $Comp
-L MXKeyboard_RGB-eagle-import:C-EUC0603K C7
-U 1 1 69A561B9
-P 14250 7100
-AR Path="/69A561B9" Ref="C7"  Part="1"
-AR Path="/5F5D6257/69A561B9" Ref="C7"  Part="1"
-F 0 "C7" V 14315 7090 59  0000 L TNN
-F 1 "0.1uF" V 14315 6990 59  0000 R TNN
-F 2 "rhais_rcl:C0603" H 14250 7100 50  0001 C CNN
-F 3 "" H 14250 7100 50  0001 C CNN
-F 4 "Multicomp" H 14250 7100 59  0001 L BNN "MFR"
-F 5 "MC0603B104J250CT" H 14250 7100 59  0001 L BNN "MPN"
-F 6 "2310559" H 14250 7100 59  0001 L BNN "OC_FARNELL"
-	1    14250 7100
-	0    -1   -1   0
-$EndComp
-$Comp
 L MXKeyboard_RGB-eagle-import:NTS0104 U12
 U 1 1 A9F22F29
@@
 $EndComp
 $Comp
-L MXKeyboard_RGB-eagle-import:C-EUC0603K C8
+L Device:C_Small C8
 U 1 1 B2598F92
-P 13500 5800
+P 13500 5900
 AR Path="/B2598F92" Ref="C8"  Part="1"
 AR Path="/5F5D6257/B2598F92" Ref="C8"  Part="1"
-F 0 "C8" H 13560 5815 59  0000 L BNN
-F 1 "0.1uF" H 13560 5615 59  0000 L BNN
-F 2 "rhais_rcl:C0603" H 13500 5800 50  0001 C CNN
-F 3 "" H 13500 5800 50  0001 C CNN
-F 4 "Multicomp" H 13500 5800 59  0001 L BNN "MFR"
-F 5 "MC0603B104J250CT" H 13500 5800 59  0001 L BNN "MPN"
-F 6 "2310559" H 13500 5800 59  0001 L BNN "OC_FARNELL"
-	1    13500 5800
-	1    0    0    -1
-$EndComp
-$Comp
-L MXKeyboard_RGB-eagle-import:C-EUC0603K C9
+F 0 "C8" H 13550 5950 59  0000 L BNN
+F 1 "0.1uF" H 13550 5850 59  0000 L TNN
+F 2 "rhais_rcl:C0603" H 13500 5900 50  0001 C CNN
+F 3 "" H 13500 5900 50  0001 C CNN
+F 4 "Multicomp" H 13500 5900 59  0001 L BNN "MFR"
+F 5 "MC0603B104J250CT" H 13500 5900 59  0001 L BNN "MPN"
+F 6 "2310559" H 13500 5900 59  0001 L BNN "OC_FARNELL"
+	1    13500 5900
+	1    0    0    -1
+$EndComp
+$Comp
+L Device:C_Small C9
 U 1 1 F7AEDC46
-P 12100 5800
+P 12100 5900
 AR Path="/F7AEDC46" Ref="C9"  Part="1"
 AR Path="/5F5D6257/F7AEDC46" Ref="C9"  Part="1"
-F 0 "C9" H 12160 5815 59  0000 L BNN
-F 1 "0.1uF" H 12160 5615 59  0000 L BNN
-F 2 "rhais_rcl:C0603" H 12100 5800 50  0001 C CNN
-F 3 "" H 12100 5800 50  0001 C CNN
-F 4 "Multicomp" H 12100 5800 59  0001 L BNN "MFR"
-F 5 "MC0603B104J250CT" H 12100 5800 59  0001 L BNN "MPN"
-F 6 "2310559" H 12100 5800 59  0001 L BNN "OC_FARNELL"
-	1    12100 5800
-	1    0    0    -1
+F 0 "C9" H 12150 5950 59  0000 L BNN
+F 1 "0.1uF" H 12150 5850 59  0000 L TNN
+F 2 "rhais_rcl:C0603" H 12100 5900 50  0001 C CNN
+F 3 "" H 12100 5900 50  0001 C CNN
+F 4 "Multicomp" H 12100 5900 59  0001 L BNN "MFR"
+F 5 "MC0603B104J250CT" H 12100 5900 59  0001 L BNN "MPN"
+F 6 "2310559" H 12100 5900 59  0001 L BNN "OC_FARNELL"
+	1    12100 5900
+	-1   0    0    -1
 $EndComp
 $Comp
@@
 L power:GND #PWR044
 U 1 1 6F6A0276
-P 9500 6600
-F 0 "#PWR044" H 9500 6350 50  0001 C CNN
-F 1 "GND" H 9505 6427 50  0000 C CNN
-F 2 "" H 9500 6600 50  0001 C CNN
-F 3 "" H 9500 6600 50  0001 C CNN
-	1    9500 6600
+P 9500 6200
+F 0 "#PWR044" H 9500 5950 50  0001 C CNN
+F 1 "GND" H 9505 6027 50  0000 C CNN
+F 2 "" H 9500 6200 50  0001 C CNN
+F 3 "" H 9500 6200 50  0001 C CNN
+	1    9500 6200
 	1    0    0    -1
 $EndComp
@@
 L power:GND #PWR049
 U 1 1 6F6A2FE1
-P 14000 7500
-F 0 "#PWR049" H 14000 7250 50  0001 C CNN
-F 1 "GND" H 14005 7327 50  0000 C CNN
-F 2 "" H 14000 7500 50  0001 C CNN
-F 3 "" H 14000 7500 50  0001 C CNN
-	1    14000 7500
+P 14100 7500
+F 0 "#PWR049" H 14100 7250 50  0001 C CNN
+F 1 "GND" H 14105 7327 50  0000 C CNN
+F 2 "" H 14100 7500 50  0001 C CNN
+F 3 "" H 14100 7500 50  0001 C CNN
+	1    14100 7500
 	1    0    0    -1
 $EndComp
@@
 L power:+3.3V #PWR047
 U 1 1 6F6A34A9
-P 12600 5500
-F 0 "#PWR047" H 12600 5350 50  0001 C CNN
-F 1 "+3.3V" H 12615 5673 50  0000 C CNN
-F 2 "" H 12600 5500 50  0001 C CNN
-F 3 "" H 12600 5500 50  0001 C CNN
-	1    12600 5500
+P 12600 5600
+F 0 "#PWR047" H 12600 5450 50  0001 C CNN
+F 1 "+3.3V" H 12615 5773 50  0000 C CNN
+F 2 "" H 12600 5600 50  0001 C CNN
+F 3 "" H 12600 5600 50  0001 C CNN
+	1    12600 5600
 	1    0    0    -1
 $EndComp
@@
 L Device:R_Small R17
 U 1 1 063E4601
-P 9700 5950
+P 9700 5900
 AR Path="/063E4601" Ref="R17"  Part="1"
 AR Path="/5F5D6257/063E4601" Ref="R17"  Part="1"
-F 0 "R17" V 9650 5950 59  0000 C BNN
-F 1 "1M" V 9750 5950 59  0000 C TNN
-F 2 "rhais_rcl:R0603" H 9700 5950 50  0001 C CNN
-F 3 "" H 9700 5950 50  0001 C CNN
-F 4 "Vishay" H 9700 5950 59  0001 L BNN "MFR"
-F 5 "CRCW08051M00FKEA" H 9700 5950 59  0001 L BNN "MPN"
-F 6 "1652946" H 9700 5950 59  0001 L BNN "OC_FARNELL"
-F 7 "" H 9700 5950 59  0001 L BNN "URL"
-F 8 "https://uk.farnell.com/vishay/crcw08051m00fkea/res-1m-1-0-125w-0805-thick-film/dp/1652946" H 9700 5950 50  0001 C CNN "URL_FARNELL"
-	1    9700 5950
-	1    0    0    -1
+F 0 "R17" V 9650 5900 59  0000 C BNN
+F 1 "1M" V 9750 5900 59  0000 C TNN
+F 2 "rhais_rcl:R0603" H 9700 5900 50  0001 C CNN
+F 3 "" H 9700 5900 50  0001 C CNN
+F 4 "Vishay" H 9700 5900 59  0001 L BNN "MFR"
+F 5 "CRCW08051M00FKEA" H 9700 5900 59  0001 L BNN "MPN"
+F 6 "1652946" H 9700 5900 59  0001 L BNN "OC_FARNELL"
+F 7 "" H 9700 5900 59  0001 L BNN "URL"
+F 8 "https://uk.farnell.com/vishay/crcw08051m00fkea/res-1m-1-0-125w-0805-thick-film/dp/1652946" H 9700 5900 50  0001 C CNN "URL_FARNELL"
+	1    9700 5900
+	1    0    0    -1
+$EndComp
+$Comp
+L Device:C_Small C7
+U 1 1 69A561B9
+P 14300 7100
+AR Path="/69A561B9" Ref="C7"  Part="1"
+AR Path="/5F5D6257/69A561B9" Ref="C7"  Part="1"
+F 0 "C7" V 14350 7150 59  0000 L CNN
+F 1 "0.1uF" V 14350 7050 59  0000 R CNN
+F 2 "rhais_rcl:C0603" H 14300 7100 50  0001 C CNN
+F 3 "" H 14300 7100 50  0001 C CNN
+F 4 "Multicomp" H 14300 7100 59  0001 L BNN "MFR"
+F 5 "MC0603B104J250CT" H 14300 7100 59  0001 L BNN "MPN"
+F 6 "2310559" H 14300 7100 59  0001 L BNN "OC_FARNELL"
+	1    14300 7100
+	0    -1   -1   0
 $EndComp
 Wire Bus Line

Commit message: Cleaned up the last capacitors that were using the eagle import schematic symbol
Parts:
- C11, C12, C13, C2, C3, C4, C5, C6: symbol MXKeyboard_RGB-eagle-import:C-EUC0603K -> Device:C_Small

Commit message: Switched the JTAG connector over to use a KiCAD + rhais part
Parts:
- JP1: footprint MXKeyboard_RGB:20021121-00010C4LF -> rhais_connector-pinheader:PinHeader_2x05_P1.27mm_Vertical_SMD; symbol MXKeyboard_RGB-eagle-import:PINHD-2X5 -> Connector_Generic:Conn_02x05_Odd_Even
- PS/2: MFR (none) -> Lumberg; MPN (none) -> TM 0508 A/6; OC_FARNELL (none) -> 1200113; URL_FARNELL (none) -> https://uk.farnell.com/lumberg/tm-0508-a-6/socket-mini-din-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
Connections:
- no-connect marks 28 -> 29
Changed lines of the file:
@@
 	5700 7500 5700 7400
 Wire Wire Line
-	3800 2400 4000 2400
+	3900 2400 4000 2400
 Wire Wire Line
 	4000 2400 4050 2400
 Wire Wire Line
-	3800 2000 4050 2000
+	3900 2000 4050 2000
 Wire Wire Line
 	4050 2400 4050 2000
@@
 	4500 5900 4400 5900
 Wire Wire Line
-	3500 2200 3300 2200
+	3400 2200 3300 2200
 Text Label 3300 2200 2    50   ~ 0
 TMS
@@
 TDI
 Wire Wire Line
-	3500 2400 3300 2400
+	3400 2400 3300 2400
 Text Label 3300 2400 2    50   ~ 0
 TDI
@@
 TCK
 Wire Wire Line
-	3500 2000 3300 2000
+	3400 2000 3300 2000
 Text Label 3300 2000 2    50   ~ 0
 TCK
@@
 TDO
 Wire Wire Line
-	3500 2100 3300 2100
+	3400 2100 3300 2100
 Text Label 3300 2100 2    50   ~ 0
 TDO
-Wire Wire Line
-	3800 2300 4000 2300
 Wire Wire Line
 	5100 4200 5100 4100
@@
 ~RESET
 Wire Wire Line
-	3800 2200 4100 2200
+	3900 2200 4100 2200
 Text Label 4100 2200 0    50   ~ 0
 ~RESET
 Wire Wire Line
-	3800 2100 4000 2100
+	3900 2100 4000 2100
 Wire Wire Line
 	4000 2100 4000 1900
@@
 $EndComp
 $Comp
-L MXKeyboard_RGB-eagle-import:PINHD-2X5 JP1
+L Connector_Generic:Conn_02x05_Odd_Even JP1
 U 1 1 2F430EF2
 P 3600 2200
@@
 F 0 "JP1" H 3350 2525 59  0000 L BNN
 F 1 "PINHD-2X5" H 3350 1800 59  0000 L BNN
-F 2 "MXKeyboard_RGB:20021121-00010C4LF" H 3600 2200 50  0001 C CNN
+F 2 "rhais_connector-pinheader:PinHeader_2x05_P1.27mm_Vertical_SMD" H 3600 2200 50  0001 C CNN
 F 3 "" H 3600 2200 50  0001 C CNN
 	1    3600 2200
@@
 F 1 "PS_2" H 14300 6300 50  0001 C CNN
 F 2 "MXKeyboard_RGB:TM_0508_A_6" H 14300 6300 50  0001 C CNN
-F 3 "" H 14300 6300 50  0001 C CNN
+F 3 "https://downloads.lumberg.com/datenblaetter/en/tm0508a.pdf" H 14300 6300 50  0001 C CNN
+F 4 "https://uk.farnell.com/lumberg/tm-0508-a-6/socket-mini-din-chassis-6-way/dp/1200113" H 14300 6300 50  0001 C CNN "URL_FARNELL"
+F 5 "1200113" H 14300 6300 50  0001 C CNN "OC_FARNELL"
+F 6 "TM 0508 A/6" H 14300 6300 50  0001 C CNN "MPN"
+F 7 "Lumberg" H 14300 6300 50  0001 C CNN "MFR"
 	1    14300 6300
 	1    0    0    -1
@@
 NoConn ~ 5500 4200
 NoConn ~ 5200 4200
-NoConn ~ 3500 2300
+NoConn ~ 3400 2300
 NoConn ~ 9300 2200
 Wire Wire Line
@@
 	0    -1   -1   0
 $EndComp
+NoConn ~ 3900 2300
 Wire Bus Line
 	4350 4400 4350 4800

Commit message: Switched the processor to use the rhais_package-qfn QFN-64 footprint
Parts:
- U11: footprint MXKeyboard_RGB:VQFN-64 -> rhais_package-qfn:QFN-64-1EP_9x9mm_P0.5mm_EP7.5x7.5mm
Changed lines of the file:
@@
 F 0 "U11" H 6800 7320 59  0000 R BNN
 F 1 "ATXMEGA256A3U-MH" H 6800 4280 59  0000 R TNN
-F 2 "MXKeyboard_RGB:VQFN-64" H 5700 5800 50  0001 C CNN
+F 2 "rhais_package-qfn:QFN-64-1EP_9x9mm_P0.5mm_EP7.5x7.5mm" H 5700 5800 50  0001 C CNN
 F 3 "" H 5700 5800 50  0001 C CNN
 	1    5700 5800
