File: board/LEDs_+_Drivers.sch (KiCad schematic (older format))
At the start: 154 parts, among them U1 TLC5947RHBT, U10 TLC5947RHBT, U18 TLC5947RHBT, U19 TLC5947RHBT, U2 TLC5947RHBT, U20 TLC5947RHBT, U21 TLC5947RHBT, U22 TLC5947RHBT, U3 TLC5947RHBT, U4 TLC5947RHBT, U5 TLC5947RHBT, U6 TLC5947RHBT, U7 TLC5947RHBT, U8 TLC5947RHBT, U9 TLC5947RHBT

Commit message: Fixed acouple of errors in the LEDs + drivers page of the schematic and switched all the current setting resistors to 15k
Parts:
- R10, R11, R12, R13, R14, R15, R16, R25, R26, R27, R28, R29, R7, R8, R9: value 9840 -> 15k; MPN MCWR06X9531FTL -> MCWR06X1502FTL; OC_FARNELL 2447452 -> 2447256; URL_FARNELL https://uk.farnell.com/multicomp-pro/mcwr06x9531ftl/res-9k5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 -> https://uk.farnell.com/multicomp/mcwr06x1502ftl/res-15k-1-0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
Connections:
- net RED31: no longer LED36.3 (C_G), U2.12 (OUT11)
- new net: LED36.3 (C_G), U2.12 (OUT11)

Commit message: Updated the footprints in the schematic having renamed all of my published libraries
Parts:
- C14, C15, C16, C17, C18, C19, C20, C21, C22, C23, C24, C25, C26, C27, C28: footprint rcl:C0603 -> rhais_rcl:C0603
- R10, R11, R12, R13, R14, R15, R16, R25, R26, R27, R28, R29, R7, R8, R9: footprint rcl:R0603 -> rhais_rcl:R0603
Changed lines of the file:
@@
 F 0 "R7" V 1150 5300 59  0000 C BNN
 F 1 "15k" V 1250 5300 59  0000 C TNN
-F 2 "rcl:R0603" H 1200 5300 50  0001 C CNN
+F 2 "rhais_rcl:R0603" H 1200 5300 50  0001 C CNN
 F 3 "" H 1200 5300 50  0001 C CNN
 F 4 "Multicomp" H 1200 5300 59  0001 L BNN "MFR"
@@
 F 0 "R8" V 1150 8600 59  0000 C BNN
 F 1 "15k" V 1250 8600 59  0000 C TNN
-F 2 "rcl:R0603" H 1200 8600 50  0001 C CNN
+F 2 "rhais_rcl:R0603" H 1200 8600 50  0001 C CNN
 F 3 "" H 1200 8600 50  0001 C CNN
 F 4 "Multicomp" H 1200 8600 59  0001 L BNN "MFR"
@@
 F 0 "R9" V 1150 11900 59  0000 C BNN
 F 1 "15k" V 1250 11900 59  0000 C TNN
-F 2 "rcl:R0603" H 1200 11900 50  0001 C CNN
+F 2 "rhais_rcl:R0603" H 1200 11900 50  0001 C CNN
 F 3 "" H 1200 11900 50  0001 C CNN
 F 4 "Multicomp" H 1200 11900 59  0001 L BNN "MFR"
@@
 F 0 "R10" V 1150 15200 59  0000 C BNN
 F 1 "15k" V 1250 15200 59  0000 C TNN
-F 2 "rcl:R0603" H 1200 15200 50  0001 C CNN
+F 2 "rhais_rcl:R0603" H 1200 15200 50  0001 C CNN
 F 3 "" H 1200 15200 50  0001 C CNN
 F 4 "Multicomp" H 1200 15200 59  0001 L BNN "MFR"
@@
 F 0 "R11" V 1150 18500 59  0000 C BNN
 F 1 "15k" V 1250 18500 59  0000 C TNN
-F 2 "rcl:R0603" H 1200 18500 50  0001 C CNN
+F 2 "rhais_rcl:R0603" H 1200 18500 50  0001 C CNN
 F 3 "" H 1200 18500 50  0001 C CNN
 F 4 "Multicomp" H 1200 18500 59  0001 L BNN "MFR"
@@
 F 0 "R12" V 19350 5300 59  0000 C BNN
 F 1 "15k" V 19450 5300 59  0000 C TNN
-F 2 "rcl:R0603" H 19400 5300 50  0001 C CNN
+F 2 "rhais_rcl:R0603" H 19400 5300 50  0001 C CNN
 F 3 "" H 19400 5300 50  0001 C CNN
 F 4 "Multicomp" H 19400 5300 59  0001 L BNN "MFR"
@@
 F 0 "R13" V 19350 8600 59  0000 C BNN
 F 1 "15k" V 19450 8600 59  0000 C TNN
-F 2 "rcl:R0603" H 19400 8600 50  0001 C CNN
+F 2 "rhais_rcl:R0603" H 19400 8600 50  0001 C CNN
 F 3 "" H 19400 8600 50  0001 C CNN
 F 4 "Multicomp" H 19400 8600 59  0001 L BNN "MFR"
@@
 F 0 "R14" V 19350 11900 59  0000 C BNN
 F 1 "15k" V 19450 11900 59  0000 C TNN
-F 2 "rcl:R0603" H 19400 11900 50  0001 C CNN
+F 2 "rhais_rcl:R0603" H 19400 11900 50  0001 C CNN
 F 3 "" H 19400 11900 50  0001 C CNN
 F 4 "Multicomp" H 19400 11900 59  0001 L BNN "MFR"
@@
 F 0 "R15" V 19350 15200 59  0000 C BNN
 F 1 "15k" V 19450 15200 59  0000 C TNN
-F 2 "rcl:R0603" H 19400 15200 50  0001 C CNN
+F 2 "rhais_rcl:R0603" H 19400 15200 50  0001 C CNN
 F 3 "" H 19400 15200 50  0001 C CNN
 F 4 "Multicomp" H 19400 15200 59  0001 L BNN "MFR"
@@
 F 0 "R16" V 19350 18500 59  0000 C BNN
 F 1 "15k" V 19450 18500 59  0000 C TNN
-F 2 "rcl:R0603" H 19400 18500 50  0001 C CNN
+F 2 "rhais_rcl:R0603" H 19400 18500 50  0001 C CNN
 F 3 "" H 19400 18500 50  0001 C CNN
 F 4 "Multicomp" H 19400 18500 59  0001 L BNN "MFR"
@@
 F 0 "R25" V 20150 5300 59  0000 C BNN
 F 1 "15k" V 20250 5300 59  0000 C TNN
-F 2 "rcl:R0603" H 20200 5300 50  0001 C CNN
+F 2 "rhais_rcl:R0603" H 20200 5300 50  0001 C CNN
 F 3 "" H 20200 5300 50  0001 C CNN
 F 4 "Multicomp" H 20200 5300 59  0001 L BNN "MFR"
@@
 F 0 "R26" V 20150 8600 59  0000 C BNN
 F 1 "15k" V 20250 8600 59  0000 C TNN
-F 2 "rcl:R0603" H 20200 8600 50  0001 C CNN
+F 2 "rhais_rcl:R0603" H 20200 8600 50  0001 C CNN
 F 3 "" H 20200 8600 50  0001 C CNN
 F 4 "Multicomp" H 20200 8600 59  0001 L BNN "MFR"
@@
 F 0 "R27" V 20150 11900 59  0000 C BNN
 F 1 "15k" V 20250 11900 59  0000 C TNN
-F 2 "rcl:R0603" H 20200 11900 50  0001 C CNN
+F 2 "rhais_rcl:R0603" H 20200 11900 50  0001 C CNN
 F 3 "" H 20200 11900 50  0001 C CNN
 F 4 "Multicomp" H 20200 11900 59  0001 L BNN "MFR"
@@
 F 0 "R28" V 20150 15200 59  0000 C BNN
 F 1 "15k" V 20250 15200 59  0000 C TNN
-F 2 "rcl:R0603" H 20200 15200 50  0001 C CNN
+F 2 "rhais_rcl:R0603" H 20200 15200 50  0001 C CNN
 F 3 "" H 20200 15200 50  0001 C CNN
 F 4 "Multicomp" H 20200 15200 59  0001 L BNN "MFR"
@@
 F 0 "R29" V 20150 18500 59  0000 C BNN
 F 1 "15k" V 20250 18500 59  0000 C TNN
-F 2 "rcl:R0603" H 20200 18500 50  0001 C CNN
+F 2 "rhais_rcl:R0603" H 20200 18500 50  0001 C CNN
 F 3 "" H 20200 18500 50  0001 C CNN
 F 4 "Multicomp" H 20200 18500 59  0001 L BNN "MFR"
@@
 F 0 "C14" H 950 4800 59  0000 L CNN
 F 1 "0.1uF" H 950 4600 59  0000 L CNN
-F 2 "rcl:C0603" H 900 4700 50  0001 C CNN
+F 2 "rhais_rcl:C0603" H 900 4700 50  0001 C CNN
 F 3 "" H 900 4700 50  0001 C CNN
 F 4 "Multicomp" H 900 4700 59  0001 L BNN "MFR"
@@
 F 0 "C15" H 19760 4615 59  0000 L BNN
 F 1 "0.1uF" H 19760 4415 59  0000 L BNN
-F 2 "rcl:C0603" H 19700 4600 50  0001 C CNN
+F 2 "rhais_rcl:C0603" H 19700 4600 50  0001 C CNN
 F 3 "" H 19700 4600 50  0001 C CNN
 F 4 "Multicomp" H 19700 4600 59  0001 L BNN "MFR"
@@
 F 0 "C16" H 19960 4615 59  0000 L BNN
 F 1 "0.1uF" H 19960 4415 59  0000 L BNN
-F 2 "rcl:C0603" H 19900 4600 50  0001 C CNN
+F 2 "rhais_rcl:C0603" H 19900 4600 50  0001 C CNN
 F 3 "" H 19900 4600 50  0001 C CNN
 F 4 "Multicomp" H 19900 4600 59  0001 L BNN "MFR"
@@
 F 0 "C17" H 950 8100 59  0000 L CNN
 F 1 "0.1uF" H 950 7900 59  0000 L CNN
-F 2 "rcl:C0603" H 900 8000 50  0001 C CNN
+F 2 "rhais_rcl:C0603" H 900 8000 50  0001 C CNN
 F 3 "" H 900 8000 50  0001 C CNN
 F 4 "Multicomp" H 900 8000 59  0001 L BNN "MFR"
@@
 F 0 "C18" H 19760 7915 59  0000 L BNN
 F 1 "0.1uF" H 19760 7715 59  0000 L BNN
-F 2 "rcl:C0603" H 19700 7900 50  0001 C CNN
+F 2 "rhais_rcl:C0603" H 19700 7900 50  0001 C CNN
 F 3 "" H 19700 7900 50  0001 C CNN
 F 4 "Multicomp" H 19700 7900 59  0001 L BNN "MFR"
@@
 F 0 "C19" H 19960 7915 59  0000 L BNN
 F 1 "0.1uF" H 19960 7715 59  0000 L BNN
-F 2 "rcl:C0603" H 19900 7900 50  0001 C CNN
+F 2 "rhais_rcl:C0603" H 19900 7900 50  0001 C CNN
 F 3 "" H 19900 7900 50  0001 C CNN
 F 4 "Multicomp" H 19900 7900 59  0001 L BNN "MFR"
@@
 F 0 "C20" H 950 11400 59  0000 L CNN
 F 1 "0.1uF" H 950 11200 59  0000 L CNN
-F 2 "rcl:C0603" H 900 11300 50  0001 C CNN
+F 2 "rhais_rcl:C0603" H 900 11300 50  0001 C CNN
 F 3 "" H 900 11300 50  0001 C CNN
 F 4 "Multicomp" H 900 11300 59  0001 L BNN "MFR"
@@
 F 0 "C21" H 19760 11215 59  0000 L BNN
 F 1 "0.1uF" H 19760 11015 59  0000 L BNN
-F 2 "rcl:C0603" H 19700 11200 50  0001 C CNN
+F 2 "rhais_rcl:C0603" H 19700 11200 50  0001 C CNN
 F 3 "" H 19700 11200 50  0001 C CNN
 F 4 "Multicomp" H 19700 11200 59  0001 L BNN "MFR"
@@
 F 0 "C22" H 19960 11215 59  0000 L BNN
 F 1 "0.1uF" H 19960 11015 59  0000 L BNN
-F 2 "rcl:C0603" H 19900 11200 50  0001 C CNN
+F 2 "rhais_rcl:C0603" H 19900 11200 50  0001 C CNN
 F 3 "" H 19900 11200 50  0001 C CNN
 F 4 "Multicomp" H 19900 11200 59  0001 L BNN "MFR"
@@
 F 0 "C23" H 900 14700 59  0000 L CNN
 F 1 "0.1uF" H 900 14500 59  0000 L CNN
-F 2 "rcl:C0603" H 850 14600 50  0001 C CNN
+F 2 "rhais_rcl:C0603" H 850 14600 50  0001 C CNN
 F 3 "" H 850 14600 50  0001 C CNN
 F 4 "Multicomp" H 850 14600 59  0001 L BNN "MFR"
@@
 F 0 "C24" H 19760 14515 59  0000 L BNN
 F 1 "0.1uF" H 19760 14315 59  0000 L BNN
-F 2 "rcl:C0603" H 19700 14500 50  0001 C CNN
+F 2 "rhais_rcl:C0603" H 19700 14500 50  0001 C CNN
 F 3 "" H 19700 14500 50  0001 C CNN
 F 4 "Multicomp" H 19700 14500 59  0001 L BNN "MFR"
@@
 F 0 "C25" H 19960 14515 59  0000 L BNN
 F 1 "0.1uF" H 19960 14315 59  0000 L BNN
-F 2 "rcl:C0603" H 19900 14500 50  0001 C CNN
+F 2 "rhais_rcl:C0603" H 19900 14500 50  0001 C CNN
 F 3 "" H 19900 14500 50  0001 C CNN
 F 4 "Multicomp" H 19900 14500 59  0001 L BNN "MFR"
@@
 F 0 "C27" H 19760 17815 59  0000 L BNN
 F 1 "0.1uF" H 19760 17615 59  0000 L BNN
-F 2 "rcl:C0603" H 19700 17800 50  0001 C CNN
+F 2 "rhais_rcl:C0603" H 19700 17800 50  0001 C CNN
 F 3 "" H 19700 17800 50  0001 C CNN
 F 4 "Multicomp" H 19700 17800 59  0001 L BNN "MFR"
@@
 F 0 "C28" H 19960 17815 59  0000 L BNN
 F 1 "0.1uF" H 19960 17615 59  0000 L BNN
-F 2 "rcl:C0603" H 19900 17800 50  0001 C CNN
+F 2 "rhais_rcl:C0603" H 19900 17800 50  0001 C CNN
 F 3 "" H 19900 17800 50  0001 C CNN
 F 4 "Multicomp" H 19900 17800 59  0001 L BNN "MFR"
@@
 F 0 "C26" H 950 18000 59  0000 L CNN
 F 1 "0.1uF" H 950 17800 59  0000 L CNN
-F 2 "rcl:C0603" H 900 17900 50  0001 C CNN
+F 2 "rhais_rcl:C0603" H 900 17900 50  0001 C CNN
 F 3 "" H 900 17900 50  0001 C CNN
 F 4 "Multicomp" H 900 17900 59  0001 L BNN "MFR"

Commit message: Fixed some silkscreen issues and flipped all the LED drivers to use a KiCAD-ified version of the LED driver schematic symbol
Parts:
- U1, U10, U18, U19, U2, U20, U21, U22, U3, U4, U5, U6, U7, U8, U9: footprint MXKeyboard_RGB:PVQFN32 -> rhais_package-qfn:VQFN-32-1EP_5x5mm_P0.5mm_EP3.5x3.5mm; symbol MXKeyboard_RGB-eagle-import:TLC5947RHBT -> DX_MON:TLC5947RHBT
Connections:
- net GND: now also U1.33 (GND), U10.33 (GND), U18.33 (GND), U19.33 (GND), U2.33 (GND), U20.33 (GND), U21.33 (GND), U22.33 (GND), U3.33 (GND), U4.33 (GND), U5.33 (GND), U6.33 (GND), U7.33 (GND), U8.33 (GND), U9.33 (GND); no longer U1.PGND (GND), U10.PGND (GND), U18.PGND (GND), U19.PGND (GND), U2.PGND (GND), U20.PGND (GND), U21.PGND (GND), U22.PGND (GND), U3.PGND (GND), U4.PGND (GND), U5.PGND (GND), U6.PGND (GND), U7.PGND (GND), U8.PGND (GND), U9.PGND (GND)

Commit message: Added BOM information for the LED drivers, cleaned up the LED schematic, and switched the LEDs over to a part that's not EOL
Parts:
- LED1, LED10, LED100, LED101, LED102, LED103, LED104, LED105, LED106, LED107, LED108, LED109, LED11, LED12, LED13, LED14, LED15, LED16, LED17, LED18, LED19, LED2, LED20, LED21, LED22, LED23, LED24, LED25, LED26, LED27, LED28, LED29, LED3, LED30, LED31, LED32, LED33, LED34, LED35, LED36, LED37, LED38, LED39, LED4, LED40, LED41, LED42, LED43, LED44, LED45, LED46, LED47, LED48, LED49, LED5, LED50, LED51, LED52, LED53, LED54, LED55, LED56, LED57, LED58, LED59, LED6, LED60, LED61, LED62, LED63, LED64, LED65, LED66, LED67, LED68, LED69, LED7, LED70, LED71, LED72, LED73, LED74, LED75, LED76, LED77, LED78, LED79, LED8, LED80, LED81, LED82, LED83, LED84, LED85, LED86, LED87, LED88, LED89, LED9, LED90, LED91, LED92, LED93, LED94, LED95, LED96, LED97, LED98, LED99: value RGB_LED-1612 -> RGB_LED-1616; footprint MXKeyboard_RGB:CHIPLED_1612 -> rhais_led:LED0606_Clockwise; symbol MXKeyboard_RGB-eagle-import:RGB_LED-1612 -> DX_MON:RGB_LED-1616; MFR (none) -> Togia LED; MPN (none) -> TJ-S1615SW6TGLCCYRGB-A5; OC_LCSC (none) -> C273610; URL_LCSC (none) -> https://lcsc.com/product-detail/Light-Emitting-Diodes-LED_T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
- R10, R11, R7, R8, R9: value 15k -> 33k; MPN MCWR06X1502FTL -> MCWR06X3302FTL; OC_FARNELL 2447256 -> 2447342; URL_FARNELL https://uk.farnell.com/multicomp/mcwr06x1502ftl/res-15k-1-0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 -> https://uk.farnell.com/multicomp/mcwr06x3302ftl/res-33k-1-0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
- U1, U10, U18, U19, U2, U20, U21, U22, U3, U4, U5, U6, U7, U8, U9: MFR (none) -> Texas Instruments; MPN (none) -> TLC5947RHBT; OC_FARNELL (none) -> 3119197; URL_FARNELL (none) -> https://uk.farnell.com/texas-instruments/tlc5947rhbt/led-dr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
Connections:
- net +5V: now also LED1.1 (A), LED10.1 (A), LED100.1 (A), LED101.1 (A), LED102.1 (A), LED103.1 (A), LED104.1 (A), LED105.1 (A), LED106.1 (A), LED107.1 (A), LED108.1 (A), LED109.1 (A), LED11.1 (A), LED12.1 (A), LED13.1 (A), LED14.1 (A), LED15.1 (A), LED16.1 (A), LED17.1 (A), LED18.1 (A), LED19.1 (A), LED2.1 (A), LED20.1 (A), LED21.1 (A), LED22.1 (A), LED23.1 (A), LED24.1 (A), LED25.1 (A), LED26.1 (A), LED27.1 (A), LED28.1 (A), LED29.1 (A), LED3.1 (A), LED30.1 (A), LED31.1 (A), LED32.1 (A), LED33.1 (A), LED34.1 (A), LED35.1 (A), LED36.1 (A), LED37.1 (A), LED38.1 (A), LED39.1 (A), LED4.1 (A), LED40.1 (A), LED41.1 (A), LED42.1 (A), LED43.1 (A), LED44.1 (A), LED45.1 (A), LED46.1 (A), LED47.1 (A), LED48.1 (A), LED49.1 (A), LED5.1 (A), LED50.1 (A), LED51.1 (A), LED52.1 (A), LED53.1 (A), LED54.1 (A), LED55.1 (A), LED56.1 (A), LED57.1 (A), LED58.1 (A), LED59.1 (A), LED6.1 (A), LED60.1 (A), LED61.1 (A), LED62.1 (A), LED63.1 (A), LED64.1 (A), LED65.1 (A), LED66.1 (A), LED67.1 (A), LED68.1 (A), LED69.1 (A), LED7.1 (A), LED70.1 (A), LED71.1 (A), LED72.1 (A), LED73.1 (A), LED74.1 (A), LED75.1 (A), LED76.1 (A), LED77.1 (A), LED78.1 (A), LED79.1 (A), LED8.1 (A), LED80.1 (A), LED81.1 (A), LED82.1 (A), LED83.1 (A), LED84.1 (A), LED85.1 (A), LED86.1 (A), LED87.1 (A), LED88.1 (A), LED89.1 (A), LED9.1 (A), LED90.1 (A), LED91.1 (A), LED92.1 (A), LED93.1 (A), LED94.1 (A), LED95.1 (A), LED96.1 (A), LED97.1 (A), LED98.1 (A), LED99.1 (A); no longer LED1.2 (A), LED10.2 (A), LED100.2 (A), LED101.2 (A), LED102.2 (A), LED103.2 (A), LED104.2 (A), LED105.2 (A), LED106.2 (A), LED107.2 (A), LED108.2 (A), LED109.2 (A), LED11.2 (A), LED12.2 (A), LED13.2 (A), LED14.2 (A), LED15.2 (A), LED16.2 (A), LED17.2 (A), LED18.2 (A), LED19.2 (A), LED2.2 (A), LED20.2 (A), LED21.2 (A), LED22.2 (A), LED23.2 (A), LED24.2 (A), LED25.2 (A), LED26.2 (A), LED27.2 (A), LED28.2 (A), LED29.2 (A), LED3.2 (A), LED30.2 (A), LED31.2 (A), LED32.2 (A), LED33.2 (A), LED34.2 (A), LED35.2 (A), LED36.2 (A), LED37.2 (A), LED38.2 (A), LED39.2 (A), LED4.2 (A), LED40.2 (A), LED41.2 (A), LED42.2 (A), LED43.2 (A), LED44.2 (A), LED45.2 (A), LED46.2 (A), LED47.2 (A), LED48.2 (A), LED49.2 (A), LED5.2 (A), LED50.2 (A), LED51.2 (A), LED52.2 (A), LED53.2 (A), LED54.2 (A), LED55.2 (A), LED56.2 (A), LED57.2 (A), LED58.2 (A), LED59.2 (A), LED6.2 (A), LED60.2 (A), LED61.2 (A), LED62.2 (A), LED63.2 (A), LED64.2 (A), LED65.2 (A), LED66.2 (A), LED67.2 (A), LED68.2 (A), LED69.2 (A), LED7.2 (A), LED70.2 (A), LED71.2 (A), LED72.2 (A), LED73.2 (A), LED74.2 (A), LED75.2 (A), LED76.2 (A), LED77.2 (A), LED78.2 (A), LED79.2 (A), LED8.2 (A), LED80.2 (A), LED81.2 (A), LED82.2 (A), LED83.2 (A), LED84.2 (A), LED85.2 (A), LED86.2 (A), LED87.2 (A), LED88.2 (A), LED89.2 (A), LED9.2 (A), LED90.2 (A), LED91.2 (A), LED92.2 (A), LED93.2 (A), LED94.2 (A), LED95.2 (A), LED96.2 (A), LED97.2 (A), LED98.2 (A), LED99.2 (A)
- net at U9.14 (OUT13): now also LED86.2 (C_B); no longer LED86.1 (C_B)
- net at U7.4 (OUT3): now also LED28.2 (C_B); no longer LED28.1 (C_B)
- net at U7.3 (OUT2): now also LED27.2 (C_B); no longer LED27.1 (C_B)
- net at U7.1 (OUT0): now also LED25.2 (C_B); no longer LED25.1 (C_B)
- net at U6.22 (OUT21): now also LED22.2 (C_B); no longer LED22.1 (C_B)
- net at U7.24 (OUT23): now also LED48.2 (C_B); no longer LED48.1 (C_B)
- net at U7.12 (OUT11): now also LED36.2 (C_B); no longer LED36.1 (C_B)
- net at U6.14 (OUT13): now also LED14.2 (C_B); no longer LED14.1 (C_B)
- net at U9.21 (OUT20): now also LED93.2 (C_B); no longer LED93.1 (C_B)
- net at U9.15 (OUT14): now also LED87.2 (C_B); no longer LED87.1 (C_B)
- net at U6.7 (OUT6): now also LED7.2 (C_B); no longer LED7.1 (C_B)
- net at U7.13 (OUT12): now also LED37.2 (C_B); no longer LED37.1 (C_B)
- net at U6.8 (OUT7): now also LED8.2 (C_B); no longer LED8.1 (C_B)
- net at U9.24 (OUT23): now also LED96.2 (C_B); no longer LED96.1 (C_B)
- net at U10.4 (OUT3): now also LED100.2 (C_B); no longer LED100.1 (C_B)
- net at U8.13 (OUT12): now also LED61.2 (C_B); no longer LED61.1 (C_B)
- net at U6.6 (OUT5): now also LED6.2 (C_B); no longer LED6.1 (C_B)
- net at U6.16 (OUT15): now also LED16.2 (C_B); no longer LED16.1 (C_B)
- net at U8.5 (OUT4): now also LED53.2 (C_B); no longer LED53.1 (C_B)
- net at U9.6 (OUT5): now also LED78.2 (C_B); no longer LED78.1 (C_B)
- net at U9.9 (OUT8): now also LED81.2 (C_B); no longer LED81.1 (C_B)
- net at U10.3 (OUT2): now also LED99.2 (C_B); no longer LED99.1 (C_B)
- net at U10.7 (OUT6): now also LED103.2 (C_B); no longer LED103.1 (C_B)
- net at U7.14 (OUT13): now also LED38.2 (C_B); no longer LED38.1 (C_B)
- net at U6.12 (OUT11): now also LED12.2 (C_B); no longer LED12.1 (C_B)
- net at U9.1 (OUT0): now also LED73.2 (C_B); no longer LED73.1 (C_B)
- net at U9.10 (OUT9): now also LED82.2 (C_B); no longer LED82.1 (C_B)
- net at U9.11 (OUT10): now also LED83.2 (C_B); no longer LED83.1 (C_B)
- net at U9.12 (OUT11): now also LED84.2 (C_B); no longer LED84.1 (C_B)
- net at U9.13 (OUT12): now also LED85.2 (C_B); no longer LED85.1 (C_B)
- net at U9.16 (OUT15): now also LED88.2 (C_B); no longer LED88.1 (C_B)
- net at U9.17 (OUT16): now also LED89.2 (C_B); no longer LED89.1 (C_B)
- net at U9.18 (OUT17): now also LED90.2 (C_B); no longer LED90.1 (C_B)
- net at U9.19 (OUT18): now also LED91.2 (C_B); no longer LED91.1 (C_B)
- net at U9.2 (OUT1): now also LED74.2 (C_B); no longer LED74.1 (C_B)
- net at U9.20 (OUT19): now also LED92.2 (C_B); no longer LED92.1 (C_B)
- net at U9.22 (OUT21): now also LED94.2 (C_B); no longer LED94.1 (C_B)
- net at U9.23 (OUT22): now also LED95.2 (C_B); no longer LED95.1 (C_B)
- net at U9.3 (OUT2): now also LED75.2 (C_B); no longer LED75.1 (C_B)
- net at U9.4 (OUT3): now also LED76.2 (C_B); no longer LED76.1 (C_B)
- net at U9.5 (OUT4): now also LED77.2 (C_B); no longer LED77.1 (C_B)
- net at U9.7 (OUT6): now also LED79.2 (C_B); no longer LED79.1 (C_B)
- net at U9.8 (OUT7): now also LED80.2 (C_B); no longer LED80.1 (C_B)
- net at U6.11 (OUT10): now also LED11.2 (C_B); no longer LED11.1 (C_B)
- net at U10.1 (OUT0): now also LED97.2 (C_B); no longer LED97.1 (C_B)
- net at U8.23 (OUT22): now also LED71.2 (C_B); no longer LED71.1 (C_B)
- net at U6.18 (OUT17): now also LED18.2 (C_B); no longer LED18.1 (C_B)
- net at U8.4 (OUT3): now also LED52.2 (C_B); no longer LED52.1 (C_B)
- net at U6.3 (OUT2): now also LED3.2 (C_B); no longer LED3.1 (C_B)
- net at U10.2 (OUT1): now also LED98.2 (C_B); no longer LED98.1 (C_B)
- net at U8.2 (OUT1): now also LED50.2 (C_B); no longer LED50.1 (C_B)
- net at U10.13 (OUT12): now also LED109.2 (C_B); no longer LED109.1 (C_B)
- net at U8.7 (OUT6): now also LED55.2 (C_B); no longer LED55.1 (C_B)
- net at U6.13 (OUT12): now also LED13.2 (C_B); no longer LED13.1 (C_B)
- net at U7.10 (OUT9): now also LED34.2 (C_B); no longer LED34.1 (C_B)
- net at U7.11 (OUT10): now also LED35.2 (C_B); no longer LED35.1 (C_B)
- net at U7.15 (OUT14): now also LED39.2 (C_B); no longer LED39.1 (C_B)
- net at U7.16 (OUT15): now also LED40.2 (C_B); no longer LED40.1 (C_B)
- net at U7.17 (OUT16): now also LED41.2 (C_B); no longer LED41.1 (C_B)
- net at U7.18 (OUT17): now also LED42.2 (C_B); no longer LED42.1 (C_B)
- net at U7.19 (OUT18): now also LED43.2 (C_B); no longer LED43.1 (C_B)
- net at U7.2 (OUT1): now also LED26.2 (C_B); no longer LED26.1 (C_B)
- net at U7.20 (OUT19): now also LED44.2 (C_B); no longer LED44.1 (C_B)
- net at U7.21 (OUT20): now also LED45.2 (C_B); no longer LED45.1 (C_B)
- net at U7.22 (OUT21): now also LED46.2 (C_B); no longer LED46.1 (C_B)
- net at U7.23 (OUT22): now also LED47.2 (C_B); no longer LED47.1 (C_B)
- net at U7.5 (OUT4): now also LED29.2 (C_B); no longer LED29.1 (C_B)
- net at U7.6 (OUT5): now also LED30.2 (C_B); no longer LED30.1 (C_B)
- net at U7.7 (OUT6): now also LED31.2 (C_B); no longer LED31.1 (C_B)
- net at U7.8 (OUT7): now also LED32.2 (C_B); no longer LED32.1 (C_B)
- net at U7.9 (OUT8): now also LED33.2 (C_B); no longer LED33.1 (C_B)
- net at U10.8 (OUT7): now also LED104.2 (C_B); no longer LED104.1 (C_B)
- net at U6.2 (OUT1): now also LED2.2 (C_B); no longer LED2.1 (C_B)
- net at U8.18 (OUT17): now also LED66.2 (C_B); no longer LED66.1 (C_B)
- net at U8.21 (OUT20): now also LED69.2 (C_B); no longer LED69.1 (C_B)
- net at U8.14 (OUT13): now also LED62.2 (C_B); no longer LED62.1 (C_B)
- net at U6.10 (OUT9): now also LED10.2 (C_B); no longer LED10.1 (C_B)
- net at U8.9 (OUT8): now also LED57.2 (C_B); no longer LED57.1 (C_B)
- net at U6.23 (OUT22): now also LED23.2 (C_B); no longer LED23.1 (C_B)
- net at U8.16 (OUT15): now also LED64.2 (C_B); no longer LED64.1 (C_B)
- net at U10.9 (OUT8): now also LED105.2 (C_B); no longer LED105.1 (C_B)
- net at U8.17 (OUT16): now also LED65.2 (C_B); no longer LED65.1 (C_B)
- net at U8.1 (OUT0): now also LED49.2 (C_B); no longer LED49.1 (C_B)
- net at U8.10 (OUT9): now also LED58.2 (C_B); no longer LED58.1 (C_B)
- net at U8.11 (OUT10): now also LED59.2 (C_B); no longer LED59.1 (C_B)
- net at U8.12 (OUT11): now also LED60.2 (C_B); no longer LED60.1 (C_B)
- net at U8.15 (OUT14): now also LED63.2 (C_B); no longer LED63.1 (C_B)
- net at U8.19 (OUT18): now also LED67.2 (C_B); no longer LED67.1 (C_B)
- net at U8.20 (OUT19): now also LED68.2 (C_B); no longer LED68.1 (C_B)
- net at U8.22 (OUT21): now also LED70.2 (C_B); no longer LED70.1 (C_B)
- net at U8.24 (OUT23): now also LED72.2 (C_B); no longer LED72.1 (C_B)
- net at U8.3 (OUT2): now also LED51.2 (C_B); no longer LED51.1 (C_B)
- net at U8.6 (OUT5): now also LED54.2 (C_B); no longer LED54.1 (C_B)
- net at U8.8 (OUT7): now also LED56.2 (C_B); no longer LED56.1 (C_B)
- net at U10.6 (OUT5): now also LED102.2 (C_B); no longer LED102.1 (C_B)
- net at U10.5 (OUT4): now also LED101.2 (C_B); no longer LED101.1 (C_B)
- net at U6.9 (OUT8): now also LED9.2 (C_B); no longer LED9.1 (C_B)
- net at U6.5 (OUT4): now also LED5.2 (C_B); no longer LED5.1 (C_B)
- net at U10.11 (OUT10): now also LED107.2 (C_B); no longer LED107.1 (C_B)
- net at U6.17 (OUT16): now also LED17.2 (C_B); no longer LED17.1 (C_B)
- net at U6.21 (OUT20): now also LED21.2 (C_B); no longer LED21.1 (C_B)
- net at U10.12 (OUT11): now also LED108.2 (C_B); no longer LED108.1 (C_B)
- net at U10.10 (OUT9): now also LED106.2 (C_B); no longer LED106.1 (C_B)
- net at U6.15 (OUT14): now also LED15.2 (C_B); no longer LED15.1 (C_B)
- net at U6.20 (OUT19): now also LED20.2 (C_B); no longer LED20.1 (C_B)
- net at U6.19 (OUT18): now also LED19.2 (C_B); no longer LED19.1 (C_B)
- net at U6.4 (OUT3): now also LED4.2 (C_B); no longer LED4.1 (C_B)
- net at U6.24 (OUT23): now also LED24.2 (C_B); no longer LED24.1 (C_B)
- net at U6.1 (OUT0): now also LED1.2 (C_B); no longer LED1.1 (C_B)
