File: board/LEDs_+_Drivers.sch (KiCad schematic (older format))
At the start: 154 parts, among them U1 TLC5947RHBT, U10 TLC5947RHBT, U18 TLC5947RHBT, U19 TLC5947RHBT, U2 TLC5947RHBT, U20 TLC5947RHBT, U21 TLC5947RHBT, U22 TLC5947RHBT, U3 TLC5947RHBT, U4 TLC5947RHBT, U5 TLC5947RHBT, U6 TLC5947RHBT, U7 TLC5947RHBT, U8 TLC5947RHBT, U9 TLC5947RHBT

Commit message: Further cleanup and added footprints for SPI termination resistors for the LED drivers as a Just In Case
Parts:
- added R39, R40, R41: DNP, rhais_rcl:R0603, symbol Device:R_Small
Connections:
- net GND: now also R39.2, R40.1, R41.1
- net SCLK_BLUE: now also R40.2
- net SCLK_GREEN: now also R39.1
- net SCLK_RED: now also R41.2
Changed lines of the file:
@@
 F 6 "2447342" H 1200 5300 59  0001 L BNN "OC_FARNELL"
 F 7 "https://uk.farnell.com/multicomp/mcwr06x3302ftl/res-33k-1-0-1w-0603-thick-film/dp/2447342" H 1200 5300 59  0001 L BNN "URL_FARNELL"
-F 8 "" H 1200 5300 50  0001 C CNN "URL"
 	1    1200 5300
 	1    0    0    -1
@@
 F 6 "2447342" H 1200 8600 59  0001 L BNN "OC_FARNELL"
 F 7 "https://uk.farnell.com/multicomp/mcwr06x3302ftl/res-33k-1-0-1w-0603-thick-film/dp/2447342" H 1200 8600 59  0001 L BNN "URL_FARNELL"
-F 8 "" H 1200 8600 50  0001 C CNN "URL"
 	1    1200 8600
 	1    0    0    -1
@@
 F 6 "2447342" H 1200 11900 59  0001 L BNN "OC_FARNELL"
 F 7 "https://uk.farnell.com/multicomp/mcwr06x3302ftl/res-33k-1-0-1w-0603-thick-film/dp/2447342" H 1200 11900 59  0001 L BNN "URL_FARNELL"
-F 8 "" H 1200 11900 50  0001 C CNN "URL"
 	1    1200 11900
 	1    0    0    -1
@@
 F 6 "2447342" H 1200 15200 59  0001 L BNN "OC_FARNELL"
 F 7 "https://uk.farnell.com/multicomp/mcwr06x3302ftl/res-33k-1-0-1w-0603-thick-film/dp/2447342" H 1200 15200 59  0001 L BNN "URL_FARNELL"
-F 8 "" H 1200 15200 50  0001 C CNN "URL"
 	1    1200 15200
 	1    0    0    -1
@@
 F 6 "2447342" H 1200 18500 59  0001 L BNN "OC_FARNELL"
 F 7 "https://uk.farnell.com/multicomp/mcwr06x3302ftl/res-33k-1-0-1w-0603-thick-film/dp/2447342" H 1200 18500 59  0001 L BNN "URL_FARNELL"
-F 8 "" H 1200 18500 50  0001 C CNN "URL"
 	1    1200 18500
 	1    0    0    -1
@@
 F 6 "2447256" H 19400 5300 59  0001 L BNN "OC_FARNELL"
 F 7 "https://uk.farnell.com/multicomp/mcwr06x1502ftl/res-15k-1-0-1w-thick-film/dp/2447256" H 19400 5300 59  0001 L BNN "URL_FARNELL"
-F 8 "" H 19400 5300 50  0001 C CNN "URL"
 	1    19400 5300
 	1    0    0    -1
@@
 F 6 "2447256" H 19400 8600 59  0001 L BNN "OC_FARNELL"
 F 7 "https://uk.farnell.com/multicomp/mcwr06x1502ftl/res-15k-1-0-1w-thick-film/dp/2447256" H 19400 8600 59  0001 L BNN "URL_FARNELL"
-F 8 "" H 19400 8600 50  0001 C CNN "URL"
 	1    19400 8600
 	1    0    0    -1
@@
 F 6 "2447256" H 19400 11900 59  0001 L BNN "OC_FARNELL"
 F 7 "https://uk.farnell.com/multicomp/mcwr06x1502ftl/res-15k-1-0-1w-thick-film/dp/2447256" H 19400 11900 59  0001 L BNN "URL_FARNELL"
-F 8 "" H 19400 11900 50  0001 C CNN "URL"
 	1    19400 11900
 	1    0    0    -1
@@
 F 6 "2447256" H 19400 15200 59  0001 L BNN "OC_FARNELL"
 F 7 "https://uk.farnell.com/multicomp/mcwr06x1502ftl/res-15k-1-0-1w-thick-film/dp/2447256" H 19400 15200 59  0001 L BNN "URL_FARNELL"
-F 8 "" H 19400 15200 50  0001 C CNN "URL"
 	1    19400 15200
 	1    0    0    -1
@@
 F 6 "2447256" H 19400 18500 59  0001 L BNN "OC_FARNELL"
 F 7 "https://uk.farnell.com/multicomp/mcwr06x1502ftl/res-15k-1-0-1w-thick-film/dp/2447256" H 19400 18500 59  0001 L BNN "URL_FARNELL"
-F 8 "" H 19400 18500 50  0001 C CNN "URL"
 	1    19400 18500
 	1    0    0    -1
@@
 F 6 "2447256" H 20200 5300 59  0001 L BNN "OC_FARNELL"
 F 7 "https://uk.farnell.com/multicomp/mcwr06x1502ftl/res-15k-1-0-1w-thick-film/dp/2447256" H 20200 5300 59  0001 L BNN "URL_FARNELL"
-F 8 "" H 20200 5300 50  0001 C CNN "URL"
 	1    20200 5300
 	1    0    0    -1
@@
 F 6 "2447256" H 20200 8600 59  0001 L BNN "OC_FARNELL"
 F 7 "https://uk.farnell.com/multicomp/mcwr06x1502ftl/res-15k-1-0-1w-thick-film/dp/2447256" H 20200 8600 59  0001 L BNN "URL_FARNELL"
-F 8 "" H 20200 8600 50  0001 C CNN "URL"
 	1    20200 8600
 	1    0    0    -1
@@
 F 6 "2447256" H 20200 11900 59  0001 L BNN "OC_FARNELL"
 F 7 "https://uk.farnell.com/multicomp/mcwr06x1502ftl/res-15k-1-0-1w-thick-film/dp/2447256" H 20200 11900 59  0001 L BNN "URL_FARNELL"
-F 8 "" H 20200 11900 50  0001 C CNN "URL"
 	1    20200 11900
 	1    0    0    -1
@@
 F 6 "2447256" H 20200 15200 59  0001 L BNN "OC_FARNELL"
 F 7 "https://uk.farnell.com/multicomp/mcwr06x1502ftl/res-15k-1-0-1w-thick-film/dp/2447256" H 20200 15200 59  0001 L BNN "URL_FARNELL"
-F 8 "" H 20200 15200 50  0001 C CNN "URL"
 	1    20200 15200
 	1    0    0    -1
@@
 F 6 "2447256" H 20200 18500 59  0001 L BNN "OC_FARNELL"
 F 7 "https://uk.farnell.com/multicomp/mcwr06x1502ftl/res-15k-1-0-1w-thick-film/dp/2447256" H 20200 18500 59  0001 L BNN "URL_FARNELL"
-F 8 "" H 20200 18500 50  0001 C CNN "URL"
 	1    20200 18500
 	1    0    0    -1
@@
 Wire Wire Line
 	11800 9500 12400 9500
+$Comp
+L Device:R_Small R?
+U 1 1 60B096E7
+P 900 17300
+AR Path="/60B096E7" Ref="R?"  Part="1"
+AR Path="/5F5D569E/60B096E7" Ref="R39"  Part="1"
+F 0 "R39" V 850 17300 59  0000 C BNN
+F 1 "DNP" V 950 17300 59  0000 C TNN
+F 2 "rhais_rcl:R0603" H 900 17300 50  0001 C CNN
+F 3 "" H 900 17300 50  0001 C CNN
+	1    900  17300
+	0    1    1    0
+$EndComp
+$Comp
+L power:GND #PWR068
+U 1 1 60B0A47A
+P 700 17400
+F 0 "#PWR068" H 700 17150 50  0001 C CNN
+F 1 "GND" H 705 17227 50  0000 C CNN
+F 2 "" H 700 17400 50  0001 C CNN
+F 3 "" H 700 17400 50  0001 C CNN
+	1    700  17400
+	1    0    0    -1
+$EndComp
+Wire Wire Line
+	800  17300 700  17300
+Wire Wire Line
+	700  17300 700  17400
+Wire Wire Line
+	1000 17300 1250 17300
+Connection ~ 1250 17300
+$Comp
+L Device:R_Small R?
+U 1 1 6115BC1E
+P 19500 17100
+AR Path="/6115BC1E" Ref="R?"  Part="1"
+AR Path="/5F5D569E/6115BC1E" Ref="R40"  Part="1"
+F 0 "R40" V 19450 17100 59  0000 C BNN
+F 1 "DNP" V 19550 17100 59  0000 C TNN
+F 2 "rhais_rcl:R0603" H 19500 17100 50  0001 C CNN
+F 3 "" H 19500 17100 50  0001 C CNN
+F 4 "Multicomp" H 19500 17100 59  0001 L BNN "MFR"
+F 5 "MCWR06X1502FTL" H 19500 17100 59  0001 L BNN "MPN"
+F 6 "2447256" H 19500 17100 59  0001 L BNN "OC_FARNELL"
+F 7 "https://uk.farnell.com/multicomp/mcwr06x1502ftl/res-15k-1-0-1w-thick-film/dp/2447256" H 19500 17100 59  0001 L BNN "URL_FARNELL"
+	1    19500 17100
+	1    0    0    -1
+$EndComp
+$Comp
+L power:GND #PWR069
+U 1 1 6115D224
+P 19800 17000
+F 0 "#PWR069" H 19800 16750 50  0001 C CNN
+F 1 "GND" H 19805 16827 50  0000 C CNN
+F 2 "" H 19800 17000 50  0001 C CNN
+F 3 "" H 19800 17000 50  0001 C CNN
+	1    19800 17000
+	1    0    0    -1
+$EndComp
+$Comp
+L Device:R_Small R?
+U 1 1 614848DA
+P 20100 17100
+AR Path="/614848DA" Ref="R?"  Part="1"
+AR Path="/5F5D569E/614848DA" Ref="R41"  Part="1"
+F 0 "R41" V 20050 17100 59  0000 C BNN
+F 1 "DNP" V 20150 17100 59  0000 C TNN
+F 2 "rhais_rcl:R0603" H 20100 17100 50  0001 C CNN
+F 3 "" H 20100 17100 50  0001 C CNN
+F 4 "Multicomp" H 20100 17100 59  0001 L BNN "MFR"
+F 5 "MCWR06X1502FTL" H 20100 17100 59  0001 L BNN "MPN"
+F 6 "2447256" H 20100 17100 59  0001 L BNN "OC_FARNELL"
+F 7 "https://uk.farnell.com/multicomp/mcwr06x1502ftl/res-15k-1-0-1w-thick-film/dp/2447256" H 20100 17100 59  0001 L BNN "URL_FARNELL"
+	1    20100 17100
+	1    0    0    -1
+$EndComp
+Wire Wire Line
+	20250 17300 20100 17300
+Wire Wire Line
+	20100 17300 20100 17200
+Connection ~ 20250 17300
+Wire Wire Line
+	19350 17300 19500 17300
+Wire Wire Line
+	19500 17300 19500 17200
+Connection ~ 19350 17300
+Wire Wire Line
+	19500 17000 19500 16900
+Wire Wire Line
+	19500 16900 19800 16900
+Wire Wire Line
+	20100 16900 20100 17000
+Wire Wire Line
+	19800 17000 19800 16900
 Wire Bus Line
 	3300 17850 10400 17850
@@
 Wire Bus Line
 	22250 3300 22250 17900
+Connection ~ 19800 16900
+Wire Wire Line
+	19800 16900 20100 16900
 $EndSCHEMATC

Commit message: Cleaned up the BOM and added all the missing BOM information I could find
Parts:
- C14, C15, C16, C17, C18, C19, C20, C21, C22, C23, C24, C25, C26, C27, C28: URL_FARNELL (none) -> https://uk.farnell.com/multicomp/mc0603b104j250ct/cap-0-1-f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
- R40, R41: MFR Multicomp -> (none); MPN MCWR06X1502FTL -> (none); OC_FARNELL 2447256 -> (none); URL_FARNELL https://uk.farnell.com/multicomp/mcwr06x1502ftl/res-15k-1-0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 -> (none)
