File: hardware/Key_matrix.kicad_sch (KiCad schematic)
At the start: 243 parts

Commit message: Improved a pile of the schematic, converting it to use KiCad schematic symbols and footprints instead of eagle imports
Parts:
- D1, D10, D11, D12, D13, D14, D15, D16, D17, D18, D19, D2, D20, D21, D22, D23, D24, D25, D26, D27, D28, D29, D3, D30, D31, D32, D33, D34, D35, D36, D37, D4, D5, D6, D7, D8, D9: symbol MXKeyboard-eagle-import:BAS16VY -> Diode:BAS16VY
- S1, S10, S100, S101, S102, S103, S104, S12, S13, S14, S15, S16, S17, S19, S2, S20, S21, S22, S23, S24, S25, S26, S27, S28, S29, S30, S31, S32, S33, S34, S35, S36, S37, S38, S40, S41, S42, S43, S44, S45, S46, S47, S48, S49, S50, S51, S52, S53, S54, S56, S57, S58, S59, S60, S61, S62, S63, S64, S65, S66, S67, S68, S69, S7, S70, S76, S77, S78, S79, S8, S80, S81, S82, S83, S84, S85, S86, S87, S88, S89, S9, S90, S91, S92, S93, S95, S96, S97, S98, S99: symbol MXKeyboard-eagle-import:CHERRY_MX_KEY_NORM -> Switch:SW_SPST
- S105, S106: symbol MXKeyboard-eagle-import:CHERRY_MX_KEY_1.45X0.7 -> Switch:SW_SPST
- S11: value \\ | -> \ |; symbol MXKeyboard-eagle-import:CHERRY_MX_KEY_NORM -> Switch:SW_SPST
- S18, S3, S55, S6, S73: symbol MXKeyboard-eagle-import:CHERRY_MX_KEY_1.1 -> Switch:SW_SPST
- S39: symbol MXKeyboard-eagle-import:CHERRY_MX_KEY_4.45 -> Switch:SW_SPST
- S4: symbol MXKeyboard-eagle-import:CHERRY_MX_KEY_1.3 -> Switch:SW_SPST
- S5: symbol MXKeyboard-eagle-import:CHERRY_MX_KEY_0.9 -> Switch:SW_SPST
- S71: value # ~~ -> # ~; symbol MXKeyboard-eagle-import:CHERRY_MX_KEY_NORM -> Switch:SW_SPST
- S72: symbol MXKeyboard-eagle-import:CHERRY_MX_KEY_2 -> Switch:SW_SPST
- S74, S94: symbol MXKeyboard-eagle-import:CHERRY_MX_KEY_0.7X1.45 -> Switch:SW_SPST
- S75: symbol MXKeyboard-eagle-import:CHERRY_MX_KEY_ENTER -> Switch:SW_SPST
Connections:
- net COLUMN1: now also D1.2 (A), D1.3 (A), D2.2 (A), D2.3 (A); no longer D1.1 (A), D1.1 (A), D2.1 (A), D2.1 (A)
- net COLUMN10: now also D18.2 (A), D18.3 (A), D19.2 (A), D19.3 (A); no longer D18.1 (A), D18.1 (A), D19.1 (A), D19.1 (A)
- net COLUMN11: now also D20.2 (A), D20.3 (A), D21.2 (A), D21.3 (A); no longer D20.1 (A), D20.1 (A), D21.1 (A), D21.1 (A)
- net COLUMN12: now also D22.2 (A), D22.3 (A), D23.2 (A), D23.3 (A); no longer D22.1 (A), D22.1 (A), D23.1 (A), D23.1 (A)
- net COLUMN13: now also D24.2 (A), D24.3 (A), D25.2 (A), D25.3 (A); no longer D24.1 (A), D24.1 (A), D25.1 (A), D25.1 (A)
- net COLUMN14: now also D26.2 (A); no longer D26.1 (A)
- net COLUMN15: now also D27.2 (A), D27.3 (A); no longer D27.1 (A), D27.1 (A)
- net COLUMN16: now also D28.2 (A), D28.3 (A), D30.2 (A), D31.2 (A); no longer D28.1 (A), D28.1 (A), D30.1 (A), D31.1 (A)
- net COLUMN17: now also D29.2 (A), D29.3 (A), D31.3 (A); no longer D29.1 (A), D29.1 (A), D31.1 (A)
- net COLUMN18: now also D32.2 (A), D32.3 (A), D33.3 (A); no longer D32.1 (A), D32.1 (A), D33.1 (A)
- net COLUMN19: now also D33.2 (A), D34.2 (A), D34.3 (A); no longer D33.1 (A), D34.1 (A), D34.1 (A)
- net COLUMN2: now also D3.2 (A), D3.3 (A), D4.2 (A), D4.3 (A); no longer D3.1 (A), D3.1 (A), D4.1 (A), D4.1 (A)
- net COLUMN20: now also D35.2 (A), D35.3 (A), D36.2 (A); no longer D35.1 (A), D35.1 (A), D36.1 (A)
- net COLUMN21: now also D37.2 (A), D37.3 (A); no longer D37.1 (A), D37.1 (A)
- net COLUMN3: now also D5.2 (A), D5.3 (A), D6.2 (A), D6.3 (A); no longer D5.1 (A), D5.1 (A), D6.1 (A), D6.1 (A)
- net COLUMN4: now also D7.2 (A), D7.3 (A), D8.2 (A); no longer D7.1 (A), D7.1 (A), D8.1 (A)
- net COLUMN5: now also D11.2 (A), D8.3 (A), D9.2 (A), D9.3 (A); no longer D11.1 (A), D8.1 (A), D9.1 (A), D9.1 (A)
- net COLUMN6: now also D10.2 (A), D10.3 (A), D11.3 (A); no longer D10.1 (A), D10.1 (A), D11.1 (A)
- net COLUMN7: now also D12.2 (A), D12.3 (A), D13.2 (A), D13.3 (A); no longer D12.1 (A), D12.1 (A), D13.1 (A), D13.1 (A)
- net COLUMN8: now also D14.2 (A), D14.3 (A), D15.2 (A); no longer D14.1 (A), D14.1 (A), D15.1 (A)
- net COLUMN9: now also D16.2 (A), D16.3 (A), D17.2 (A); no longer D16.1 (A), D16.1 (A), D17.1 (A)
- net GND: now also D15.3 (A), D15.4 (K), D17.3 (A), D17.4 (K), D26.3 (A), D26.4 (K), D30.3 (A), D30.4 (K), D36.3 (A), D36.4 (K); no longer D15.1 (A), D15.6 (C), D17.1 (A), D17.6 (C), D26.1 (A), D26.6 (C), D30.1 (A), D30.6 (C), D36.1 (A), D36.6 (C)
- net at S25.2 (B): now also D9.5 (K); no longer D9.6 (C)
- net at S26.2 (B): now also D9.4 (K); no longer D9.6 (C)
- net at S77.2 (B): now also D27.5 (K); no longer D27.6 (C)
- net at S11.2 (B): now also D4.5 (K); no longer D4.6 (C)
- net at S38.2 (B): now also D13.5 (K); no longer D13.6 (C)
- net at S58.2 (B): now also D20.4 (K); no longer D20.6 (C)
- net at S17.2 (B): now also D6.5 (K); no longer D6.6 (C)
- net at S18.2 (B): now also D6.4 (K); no longer D6.6 (C)
- net at S27.2 (B): now also D11.5 (K); no longer D11.6 (C)
- net at S21.2 (B): now also D7.4 (K); no longer D7.6 (C)
- net at S42.2 (B): now also D14.4 (K); no longer D14.6 (C)
- net at S41.2 (B): now also D14.5 (K); no longer D14.6 (C)
- net at S89.2 (B): now also D31.4 (K); no longer D31.6 (C)
- net at S84.2 (B): now also D30.5 (K); no longer D30.6 (C)
- net at S39.2 (B): now also D13.4 (K); no longer D13.6 (C)
- net at S6.2 (B): now also D2.4 (K); no longer D2.6 (C)
- net at S5.2 (B): now also D2.5 (K); no longer D2.6 (C)
- net at S49.2 (B): now also D17.5 (K); no longer D17.6 (C)
- net at S20.2 (B): now also D7.5 (K); no longer D7.6 (C)
- net at S35.2 (B): now also D12.5 (K); no longer D12.6 (C)
- net at S36.2 (B): now also D12.4 (K); no longer D12.6 (C)
- net at S101.2 (B): now also D35.4 (K); no longer D35.6 (C)
- net at S44.2 (B): now also D15.5 (K); no longer D15.6 (C)
- net at S46.2 (B): now also D16.5 (K); no longer D16.6 (C)
- net at S47.2 (B): now also D16.4 (K); no longer D16.6 (C)
- net at S82.2 (B): now also D28.4 (K); no longer D28.6 (C)
- net at S100.2 (B): now also D35.5 (K); no longer D35.6 (C)
- net at S91.2 (B): now also D32.5 (K); no longer D32.6 (C)
- net at S28.2 (B): now also D8.4 (K); no longer D8.6 (C)
- net at S97.2 (B): now also D34.4 (K); no longer D34.6 (C)
- net at S9.2 (B): now also D3.4 (K); no longer D3.6 (C)
- net at S8.2 (B): now also D3.5 (K); no longer D3.6 (C)
- net at S67.2 (B): now also D23.4 (K); no longer D23.6 (C)
- net at S66.2 (B): now also D23.5 (K); no longer D23.6 (C)
- net at S92.2 (B): now also D32.4 (K); no longer D32.6 (C)
- net at S57.2 (B): now also D20.5 (K); no longer D20.6 (C)
- net at S30.2 (B): now also D10.5 (K); no longer D10.6 (C)
- net at S31.2 (B): now also D10.4 (K); no longer D10.6 (C)
- net at S61.2 (B): now also D21.4 (K); no longer D21.6 (C)
- net at S78.2 (B): now also D27.4 (K); no longer D27.6 (C)
- net at S72.2 (B): now also D25.5 (K); no longer D25.6 (C)
- net at S73.2 (B): now also D25.4 (K); no longer D25.6 (C)
- net at S69.2 (B): now also D24.5 (K); no longer D24.6 (C)
- net at S70.2 (B): now also D24.4 (K); no longer D24.6 (C)
- net at S64.2 (B): now also D22.4 (K); no longer D22.6 (C)
- net at S63.2 (B): now also D22.5 (K); no longer D22.6 (C)
- net at S33.2 (B): now also D11.4 (K); no longer D11.6 (C)
- net at S54.2 (B): now also D19.5 (K); no longer D19.6 (C)
- net at S14.2 (B): now also D5.5 (K); no longer D5.6 (C)
- net at S15.2 (B): now also D5.4 (K); no longer D5.6 (C)
- net at S103.2 (B): now also D36.5 (K); no longer D36.6 (C)
- net at S2.2 (B): now also D1.5 (K); no longer D1.6 (C)
- net at S88.2 (B): now also D29.4 (K); no longer D29.6 (C)
- net at S87.2 (B): now also D29.5 (K); no longer D29.6 (C)
- net at S98.2 (B): now also D33.5 (K); no longer D33.6 (C)
- net at S23.2 (B): now also D8.5 (K); no longer D8.6 (C)
- net at S12.2 (B): now also D4.4 (K); no longer D4.6 (C)
- net at S3.2 (B): now also D1.4 (K); no longer D1.6 (C)
- net at S96.2 (B): now also D34.5 (K); no longer D34.6 (C)
- net at S52.2 (B): now also D18.4 (K); no longer D18.6 (C)
- net at S105.2 (B): now also D37.5 (K); no longer D37.6 (C)
- net at S106.2 (B): now also D37.4 (K); no longer D37.6 (C)
- net at S85.2 (B): now also D31.5 (K); no longer D31.6 (C)
- net at S81.2 (B): now also D28.5 (K); no longer D28.6 (C)
- net at S75.2 (B): now also D26.5 (K); no longer D26.6 (C)
- net at S55.2 (B): now also D19.4 (K); no longer D19.6 (C)
- net at S51.2 (B): now also D18.5 (K); no longer D18.6 (C)
- net at S60.2 (B): now also D21.5 (K); no longer D21.6 (C)
- net at S94.2 (B): now also D33.4 (K); no longer D33.6 (C)
Other:
- moved on the sheet: R1, R2, R3, R30, R31, R32, R33, R34, R35, R4, R5, R6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
