File: hardware/LEDs_+_Drivers.kicad_sch (KiCad schematic)
At the start: 157 parts, among them U1 TLC5947RHBT, U10 TLC5947RHBT, U18 TLC5947RHBT, U19 TLC5947RHBT, U2 TLC5947RHBT, U20 TLC5947RHBT, U21 TLC5947RHBT, U22 TLC5947RHBT, U3 TLC5947RHBT, U4 TLC5947RHBT, U5 TLC5947RHBT, U6 TLC5947RHBT, U7 TLC5947RHBT, U8 TLC5947RHBT, U9 TLC5947RHBT

Commit message: Improved a pile of the schematic, converting it to use KiCad schematic symbols and footprints instead of eagle imports
Connections:
- net MOSI_BLUE renamed COPI_BLUE
- net MOSI_GREEN renamed COPI_GREEN
- net MOSI_RED renamed COPI_RED

Commit message: More work on the schematics for the keyboard, including fixing all the page sizes after a mishap
Other:
- moved on the sheet: C14, C15, C16, C17, C18, C19, C20, C21, C22, C23, C24, C25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
